File: woagpad.kicad_pcb (KiCad board)
At the start: 2 copper layers, 1 part, among them U1 XIAO-RP2040-DIP

Commit message: feat: finish schematic
Parts:
- added D1: D, ScottoKeebs_Components:Diode_DO-35, F.Cu at (76.5, 85.0)
- added D10: D, ScottoKeebs_Components:Diode_DO-35, F.Cu at (76.5, 109.8)
- added D11: D, ScottoKeebs_Components:Diode_DO-35, F.Cu at (76.5, 113.4)
- added D2: D, ScottoKeebs_Components:Diode_DO-35, F.Cu at (76.5, 88.5)
- added D3: D, ScottoKeebs_Components:Diode_DO-35, F.Cu at (76.5, 92.1)
- added D5: D, ScottoKeebs_Components:Diode_DO-35, F.Cu at (76.5, 95.6)
- added D6: D, ScottoKeebs_Components:Diode_DO-35, F.Cu at (76.5, 99.2)
- added D7: D, ScottoKeebs_Components:Diode_DO-35, F.Cu at (76.5, 102.7)
- added D9: D, ScottoKeebs_Components:Diode_DO-35, F.Cu at (76.5, 106.3)
- added J1: Conn_01x04, ScottoKeebs_Components:OLED_128x64, F.Cu at (102.3, 84.8)
- added SW10: SW_Push, ScottoKeebs_MX:MX_PCB_1.00u, F.Cu at (67.1, 106.5)
- added SW11: SW_Push, ScottoKeebs_MX:MX_PCB_1.00u, F.Cu at (67.1, 122.1)
- added SW17: RotaryEncoder_Switch, ScottoKeebs_Scotto:Encoder_EC11_MX, F.Cu at (83.9, 122.2)
- added SW18: RotaryEncoder_Switch, ScottoKeebs_Scotto:Encoder_EC11_MX, F.Cu at (83.9, 136.4)
- added SW2: SW_Push, ScottoKeebs_MX:MX_PCB_1.00u, F.Cu at (51.6, 91.0)
- added SW3: SW_Push, ScottoKeebs_MX:MX_PCB_1.00u, F.Cu at (51.6, 106.5)
- added SW5: SW_Push, ScottoKeebs_MX:MX_PCB_1.00u, F.Cu at (51.6, 122.1)
- added SW6: SW_Push, ScottoKeebs_MX:MX_PCB_1.00u, F.Cu at (51.6, 137.6)
- added SW7: SW_Push, ScottoKeebs_MX:MX_PCB_1.00u, F.Cu at (67.1, 91.0)
- U1: footprint XIAO_PCB:MOUDLE14P-2.54-21X17.8MM -> ScottoKeebs_MCU:Seeed_XIAO_RP2040
- moved U1 27.0 mm to (102.4, 68.9), turned to 0 degrees
Connections:
- U1 pad 12: unconnected-(U1-3V3-Pad12) -> VCC
- U1 pad 5: unconnected-(U1-GPIO6/SDA-Pad5) -> SDA
- U1 pad 6: unconnected-(U1-GPIO7/SCL-Pad6) -> SCL

Commit message: feat: woagpad V0.1 PCB done
Parts:
- removed D10, D11: D, ScottoKeebs_Components:Diode_DO-35
- removed SW10, SW11: SW_Push, ScottoKeebs_MX:MX_PCB_1.00u
- removed SW17, SW18: RotaryEncoder_Switch, ScottoKeebs_Scotto:Encoder_EC11_MX
- added D4: D, ScottoKeebs_Components:Diode_DO-35, B.Cu at (200.5, 87.5)
- added D8: D, ScottoKeebs_Components:Diode_DO-35, B.Cu at (219.8, 106.5)
- added MP: MountingHole_3.2mm_M3, MountingHole:MountingHole_3.2mm_M3, F.Cu at (233.4, 111.8)
- added MP: MountingHole_3.2mm_M3, MountingHole:MountingHole_3.2mm_M3, F.Cu at (241.5, 45.5)
- added MP: MountingHole_3.2mm_M3, MountingHole:MountingHole_3.2mm_M3, F.Cu at (214.4, 111.8)
- added MP: MountingHole_3.2mm_M3, MountingHole:MountingHole_3.2mm_M3, F.Cu at (206.5, 45.2)
- added QR*****: WobblQR, Library:WobblQR, F.Cu at (223.8, 34.8)
- added SW1: RotaryEncoder_Switch_MP, ScottoKeebs_Scotto:Encoder_EC11_MX, F.Cu at (205.0, 59.0)
- added SW4: SW_Push, ScottoKeebs_MX:MX_PCB, F.Cu at (205.0, 78.0)
- added SW8: SW_Push, ScottoKeebs_MX:MX_PCB, F.Cu at (224.0, 97.0)
- added SW9: SW_Push, ScottoKeebs_MX:MX_PCB, F.Cu at (243.0, 97.0)
- added kibuzzard-67AA371A: G***, kibuzzard-67AA371A, F.Cu at (224.0, 27.0)
- D1, D2, D3, D5, D6, D7, D9, U1: moved to B.Cu
- J1: value Conn_01x04 -> OLED_128x64; footprint ScottoKeebs_Components:OLED_128x64 -> Library:MODULE_DM-OLED096-636
- SW2, SW5, SW6, SW7: footprint ScottoKeebs_MX:MX_PCB_1.00u -> ScottoKeebs_MX:MX_PCB
- SW3: value SW_Push -> RotaryEncoder_Switch_MP; footprint ScottoKeebs_MX:MX_PCB_1.00u -> ScottoKeebs_Scotto:Encoder_EC11_MX
- moved SW6 200.5 mm to (243.0, 78.0)
- moved SW3 197.2 mm to (243.0, 59.0), turned to 180 degrees
- moved SW5 178.0 mm to (224.0, 78.0)
- moved SW2 175.4 mm to (224.0, 59.0)
- moved D3 164.4 mm to (239.2, 68.5)
- moved D9 162.3 mm to (238.8, 106.5)
- moved D6 162.2 mm to (238.2, 87.5)
- moved D2 144.3 mm to (219.4, 68.5)
- moved D5 143.0 mm to (219.2, 87.5)
- moved SW7 138.0 mm to (205.0, 97.0)
- moved D1 133.5 mm to (209.0, 68.5), turned to 180 degrees
- moved J1 131.1 mm to (224.0, 36.0), turned to 180 degrees
- moved U1 126.3 mm to (224.0, 34.8), turned to 180 degrees
- moved D7 123.5 mm to (199.9, 106.5)
Connections:
- D1 pad 2: E11_R0_L -> Net-(D1-A)
- D2 pad 1: R1 -> R0
- D3 pad 1: R2 -> R0
- D5 pad 1: R0 -> R1
- D9 pad 1: R0 -> R2
- D9 pad 2: E11_R0_R -> Net-(D9-A)
- SW2 pad 1: C0 -> C1
- SW6 pad 1: C1 -> C2
- SW7 pad 1: C1 -> C0
- U1 pad 1: unconnected-(U1-GPIO26/ADC0/A0-Pad1) -> ENC_R
- U1 pad 10: unconnected-(U1-GPIO4/MISO-Pad10) -> ENC_SHARED
- U1 pad 11: unconnected-(U1-GPIO3/MOSI-Pad11) -> ENC_L
- U1 pad 2: unconnected-(U1-GPIO27/ADC1/A1-Pad2) -> C2
- U1 pad 3: unconnected-(U1-GPIO28/ADC2/A2-Pad3) -> R0
- U1 pad 4: unconnected-(U1-GPIO29/ADC3/A3-Pad4) -> C1
- U1 pad 7: unconnected-(U1-GPIO0/TX-Pad7) -> R1
- U1 pad 8: unconnected-(U1-GPIO1/RX-Pad8) -> R2
- U1 pad 9: unconnected-(U1-GPIO2/SCK-Pad9) -> C0
Routing:
- net R2: track 0.00 -> 107.8 mm, vias 0 -> 1
- net R1: track 0.00 -> 88.9 mm
- net R0: track 0.00 -> 75.4 mm
- net C2: track 0.00 -> 73.6 mm
- net C1: track 0.00 -> 72.3 mm
- net C0: track 0.00 -> 70.0 mm
- net ENC_SHARED: track 0.00 -> 67.9 mm
- net ENC_R: track 0.00 -> 45.6 mm
- net ENC_L: track 0.00 -> 26.7 mm
- net Net-(D3-A): track 0.00 -> 21.2 mm
- net VCC: track 0.00 -> 19.0 mm
- net SDA: track 0.00 -> 15.7 mm
- net Net-(D5-A): track 0.00 -> 15.0 mm
- net Net-(D7-A): track 0.00 -> 15.0 mm
- net Net-(D2-A): track 0.00 -> 15.0 mm
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- added copper zone on B.Cu, net GND
- added copper zone on F.Cu, net GND
Other:
- board outline added: 57.8 x 93.5 mm
- board text added: "By Suya"
- board text added: "wobbl.in"
