File: woagpad.kicad_sch (KiCad schematic)
At the start: 33 parts, among them SW1 SW_Push, SW10 SW_Push, SW11 SW_Push, SW12 SW_Push, SW13 SW_Push, SW14 SW_Push, SW15 SW_Push, SW16 SW_Push, SW2 SW_Push, SW3 SW_Push, SW4 SW_Push, SW5 SW_Push, SW6 SW_Push, SW7 SW_Push, SW8 SW_Push, SW9 SW_Push, U1 XIAO-RP2040-DIP

Commit message: feat: finish schematic
Parts:
- removed D12, D13, D14, D15, D16, D4, D8: D, symbol Device:D_Small
- removed SW1, SW12, SW13, SW14, SW15, SW16, SW4, SW8, SW9: SW_Push, symbol Switch:SW_Push_45deg
- added J1: Conn_01x04, ScottoKeebs_Components:OLED_128x64, symbol Connector_Generic:Conn_01x04
- added SW17, SW18: RotaryEncoder_Switch, ScottoKeebs_Scotto:Encoder_EC11_MX, symbol Device:RotaryEncoder_Switch
- D1, D10, D11, D2, D3, D5, D6, D7, D9: footprint (none) -> ScottoKeebs_Components:Diode_DO-35
- SW10, SW11, SW2, SW3, SW5, SW6, SW7: footprint (none) -> ScottoKeebs_MX:MX_PCB_1.00u
- U1: footprint XIAO_PCB:MOUDLE14P-2.54-21X17.8MM -> ScottoKeebs_MCU:Seeed_XIAO_RP2040
Connections:
- net C0: now also SW17.S1
- net C2: now also SW18.S1
- net GND: now also J1.1 (Pin_1), SW17.C, SW18.C
- net E11_R0_R: now reaches D9.2 (A)
- net E11_R0_R: now also SW18.S2
- net VCC: now reaches U1.12 (3V3)
- net VCC: now also J1.2 (Pin_2)
- net SDA: now reaches U1.5 (GPIO6/SDA)
- net SDA: now also J1.4 (Pin_4)
- net SCL: now reaches U1.6 (GPIO7/SCL)
- net SCL: now also J1.3 (Pin_3)
- net E11_R0_L: now reaches D1.2 (A)
- net E11_R0_L: now also SW17.S2
- new net ENC_L: SW17.B
- new net ENC_R: SW18.B
- new net ENC_SHARED: SW17.A, SW18.A

Commit message: feat: woagpad V0.1 PCB done
Parts:
- removed J1: Conn_01x04, ScottoKeebs_Components:OLED_128x64, symbol Connector_Generic:Conn_01x04
- removed SW17, SW18: RotaryEncoder_Switch, ScottoKeebs_Scotto:Encoder_EC11_MX, symbol Device:RotaryEncoder_Switch
- added J1: OLED_128x64, Library:MODULE_DM-OLED096-636, symbol ScottoKeebs:OLED_128x64
- added SW1, SW3: RotaryEncoder_Switch_MP, ScottoKeebs_Scotto:Encoder_EC11_MX, symbol Device:RotaryEncoder_Switch_MP
- SW2: renamed from SW5; footprint ScottoKeebs_MX:MX_PCB_1.00u -> ScottoKeebs_MX:MX_PCB
- SW4: renamed from SW2; footprint ScottoKeebs_MX:MX_PCB_1.00u -> ScottoKeebs_MX:MX_PCB
- SW5: renamed from SW6; footprint ScottoKeebs_MX:MX_PCB_1.00u -> ScottoKeebs_MX:MX_PCB
- SW6: renamed from SW10; footprint ScottoKeebs_MX:MX_PCB_1.00u -> ScottoKeebs_MX:MX_PCB
- SW7: renamed from SW3; footprint ScottoKeebs_MX:MX_PCB_1.00u -> ScottoKeebs_MX:MX_PCB
- SW8: renamed from SW7; footprint ScottoKeebs_MX:MX_PCB_1.00u -> ScottoKeebs_MX:MX_PCB
- SW9: renamed from SW11; footprint ScottoKeebs_MX:MX_PCB_1.00u -> ScottoKeebs_MX:MX_PCB
- renumbered D5 to D2, D9 to D3, D2 to D4, D6 to D5, D10 to D6, D3 to D7, D7 to D8, D11 to D9
Connections:
- net C0: now also U1.9 (GPIO2/SCK), SW1.S2
- net C1: now also U1.4 (GPIO29/ADC3/A3)
- net C2: now also U1.2 (GPIO27/ADC1/A1), SW3.S2
- net ENC_L: now also U1.11 (GPIO3/MOSI), SW1.B
- net ENC_R: now also U1.1 (GPIO26/ADC0/A0), SW3.B
- net ENC_SHARED: now also U1.10 (GPIO4/MISO), SW1.A, SW3.A
- net GND: now also J1.1 (GND), SW1.C, SW1.MP, SW3.C, SW3.MP
- net R0: now also U1.3 (GPIO28/ADC2/A2)
- net R1: now also U1.7 (GPIO0/TX)
- net R2: now also U1.8 (GPIO1/RX)
- net SCL: now also J1.3 (SCL)
- net SDA: now also J1.4 (SDA)
- net VCC: now also J1.2 (VCC)
- net E11_R0_L: no longer names the net of D1.2 (A)
- net E11_R0_L: now also SW1.S1
- net E11_R0_R: no longer names the net of D3.2 (A)
- net E11_R0_R: now also SW3.S1
Other:
- moved on the sheet: D1, D2, D3, D4, D5, D6, D7, D8, D9, SW2, SW4, SW5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
